Commit message: mapping added

File: frankenstein_description/urdf/frankenstein.urdf (robot description, URDF)
Before this commit: robot frankenstein_reality, 16 links, 15 joints
Links:
- link front_right_wheel: geometry visual cylinder length=0.05 radius=0.1
- link left_free_wheel: geometry visual cylinder length=0.05 radius=0.1
- link lidar_link: geometry visual cylinder length=0.224 radius=0.06
- link rod: geometry visual box size=0.145 0.742 1.2
Joints:
- joint front_right_steering_joint: origin xyz=-0.388 0.267 -0.3759975 rpy=1.570796 0 0 -> xyz=-0.388 0.2 -0.3759975 rpy=1.570796 0 0
- joint left_free_steering_joint: origin xyz=-0.388 -0.267 -0.3759975 rpy=1.570796 0 0 -> xyz=-0.388 -0.2 -0.3759975 rpy=1.570796 0 0
- joint lidar_to_rod: origin xyz=0 0 0.695068 rpy=0 0 3.141593 -> xyz=0 0 0.623409 rpy=0 0 3.141593
- joint rod_to_chassis: origin xyz=0.3305 0 1.1075655 rpy=0 0 0 -> xyz=0.1295 0 1.0159975 rpy=0 0 0
